Commit message: gazebo_load_baseline with errors in ign plugin

File: install/kuka_description/share/kuka_description/urdf/kr150_2_macro.xacro (robot description, xacro)
@@ -2,5 +2,5 @@
 <robot xmlns:xacro="http://wiki.ros.org/xacro" name="kuka_kr150_2_robot">
   <!-- Start GZ or Ignition depending on ROS 2 Version -->
-  <xacro:arg name="is_ignition" default="true"/>
+  <xacro:arg name="is_ignition" default="False"/>
   <!-- Include Gazebo Parameters -->
   <xacro:include filename="$(find kuka_description)/urdf/kr150_gazebo.xacro" />

File: install/kuka_description/share/kuka_description/urdf/kr150_gazebo.xacro (robot description, xacro)
@@ -1,18 +1,18 @@
 <?xml version="1.0"?>
-<robot xmlns:xacro="http://www.ros.org/wiki/xacro" name="arduinobot">
-  <!-- ROS 2 Control -->
-  <gazebo>
-    <!-- ROS 2 Humble -->
+<robot xmlns:xacro="http://www.ros.org/wiki/xacro" name="kuka_kr150_2_robot">
+<gazebo>
+  <!-- Humble + Ignition -->
     <xacro:if value="$(arg is_ignition)">
       <plugin filename="ign_ros2_control-system" name="ign_ros2_control::IgnitionROS2ControlPlugin">
-        <parameters>$(find arduinobot_controller)/config/arduinobot_controllers.yaml</parameters>
+        <parameters>$(find kuka_controller)/config/kukarobot_controllers.yaml</parameters>
       </plugin>
     </xacro:if>
-    <!-- ROS 2 Iron or above -->
-    <xacro:unless value="$(arg is_ignition)">
-      <plugin filename="gz_ros2_control-system" name="gz_ros2_control::GazeboSimROS2ControlPlugin">
-        <parameters>$(find arduinobot_controller)/config/arduinobot_controllers.yaml</parameters>
-      </plugin>
-    </xacro:unless>
-  </gazebo>
+  <!-- Iron/Jazzy + Gazebo (Harmonic+) -->
+  <xacro:unless value="$(arg is_ignition)">
+    <plugin filename="libgz_ros2_control-system.so"
+            name="gz_ros2_control::GazeboSimROS2ControlPlugin">
+      <parameters>$(find kukarobot_controller)/config/kukarobot_controller.yaml</parameters>
+    </plugin>
+  </xacro:unless>
+</gazebo>
 </robot>

File: src/Kuka_description/urdf/kr150_gazebo.xacro (robot description, xacro)
@@ -1,18 +1,18 @@
 <?xml version="1.0"?>
 <robot xmlns:xacro="http://www.ros.org/wiki/xacro" name="kuka_kr150_2_robot">
-  <!-- ROS 2 Control -->
-  <gazebo>
-    <!-- ROS 2 Humble -->
+<gazebo>
+  <!-- Humble + Ignition -->
     <xacro:if value="$(arg is_ignition)">
       <plugin filename="ign_ros2_control-system" name="ign_ros2_control::IgnitionROS2ControlPlugin">
-        <parameters>$(find kukarobot_controller)/config/kukarobot_controller.yaml</parameters>
+        <parameters>$(find kuka_controller)/config/kukarobot_controllers.yaml</parameters>
       </plugin>
     </xacro:if>
-    <!-- ROS 2 Iron or above -->
-    <xacro:unless value="$(arg is_ignition)">
-      <plugin filename="gz_ros2_control-system" name="gz_ros2_control::GazeboSimROS2ControlPlugin">
-        <parameters>$(find kukarobot_controller)/config/kukarobot_controller.yaml</parameters>
-      </plugin>
-    </xacro:unless>
-  </gazebo>
+  <!-- Iron/Jazzy + Gazebo (Harmonic+) -->
+  <xacro:unless value="$(arg is_ignition)">
+    <plugin filename="libgz_ros2_control-system.so"
+            name="gz_ros2_control::GazeboSimROS2ControlPlugin">
+      <parameters>$(find kukarobot_controller)/config/kukarobot_controller.yaml</parameters>
+    </plugin>
+  </xacro:unless>
+</gazebo>
 </robot>

File: src/Kuka_description/urdf/kr150_ros2_control.xacro (robot description, xacro)
@@ -1,51 +1,73 @@
 <?xml version="1.0"?>
 <robot xmlns:xacro="http://www.ros.org/wiki/xacro" name="kuka_kr150_2_robot">
-    <ros2_control name="RobotSystem" type="system">
-        <xacro:property name="PI" value="3.14159265359" />
-        <!-- ros2_control Gazebo -->
-        <!-- ROS 2 Humble -->
-        <xacro:if value="$(arg is_ignition)">
-            <hardware>
-                <plugin>ign_ros2_control/IgnitionSystem</plugin>
-            </hardware>
-        </xacro:if>
-        <!-- ROS 2 Iron or above -->
-        <xacro:unless value="$(arg is_ignition)">
-            <hardware>
-                <plugin>gz_ros2_control/GazeboSimSystem</plugin>
-            </hardware>
-        </xacro:unless>
-        <joint name="joint_1">
-            <command_interface name="position">
-            <param name="min">-${PI / 2}</param>
-            <param name="max">${PI / 2}</param>
-            </command_interface>
-            <state_interface name="position"/>
-        </joint>
-        <joint name="joint_2">
-            <command_interface name="position">
-            <param name="min">-${PI / 2}</param>
-            <param name="max">${PI / 2}</param>
-            </command_interface>
-            <state_interface name="position"/>
-        </joint>
-        <joint name="joint_3">
-            <command_interface name="position">
-            <param name="min">-${PI / 2}</param>
-            <param name="max">${PI / 2}</param>
-            </command_interface>
-            <state_interface name="position"/>
-        </joint>
-        <joint name="joint_4">
-            <command_interface name="position">
-            <param name="min">-${PI / 2}</param>
-            <param name="max">0.0</param>
-            </command_interface>
-            <state_interface name="position"/>
-        </joint>
-        <joint name="joint_5">
-            <param name="mimic">joint_4</param>
-            <param name="multiplier">-1</param>
-        </joint>
-    </ros2_control>
+<!-- ros2_control hardware + interfaces for KR150-2 -->
+<ros2_control name="KR150System" type="system">
+  <!-- Select hardware plugin by simulator -->
+  <!-- Humble + Ignition (Fortress/Garden): ign_ros2_control -->
+  <xacro:if value="$(arg is_ignition)">
+    <hardware>
+      <plugin>ign_ros2_control/IgnitionSystem</plugin>
+    </hardware>
+  </xacro:if>
+  <!-- Iron/Jazzy/Rolling + modern Gazebo (Harmonic+): gz_ros2_control -->
+  <xacro:unless value="$(arg is_ignition)">
+    <hardware>
+      <plugin>gz_ros2_control/GazeboSimSystem</plugin>
+    </hardware>
+  </xacro:unless>
+  <!-- a1 -->
+  <joint name="joint_a1">
+    <command_interface name="position">
+      <param name="min">-3.228859116</param>
+      <param name="max"> 3.228859116</param>
+    </command_interface>
+    <state_interface name="position"/>
+    <state_interface name="velocity"/>
+  </joint>
+  <!-- a2 -->
+  <joint name="joint_a2">
+    <command_interface name="position">
+      <param name="min">-2.548180708</param>
+      <param name="max"> 0.0</param>
+    </command_interface>
+    <state_interface name="position"/>
+    <state_interface name="velocity"/>
+  </joint>
+  <!-- a3 -->
+  <joint name="joint_a3">
+    <command_interface name="position">
+      <param name="min">-2.076941810</param>
+      <param name="max"> 2.705260341</param>
+    </command_interface>
+    <state_interface name="position"/>
+    <state_interface name="velocity"/>
+  </joint>
+  <!-- a4 -->
+  <joint name="joint_a4">
+    <command_interface name="position">
+      <param name="min">-6.108652382</param>
+      <param name="max"> 6.108652382</param>
+    </command_interface>
+    <state_interface name="position"/>
+    <state_interface name="velocity"/>
+  </joint>
+  <!-- a5 -->
+  <joint name="joint_a5">
+    <command_interface name="position">
+      <param name="min">-2.181661565</param>
+      <param name="max"> 2.181661565</param>
+    </command_interface>
+    <state_interface name="position"/>
+    <state_interface name="velocity"/>
+  </joint>
+  <!-- a6 -->
+  <joint name="joint_a6">
+    <command_interface name="position">
+      <param name="min">-6.108652382</param>
+      <param name="max"> 6.108652382</param>
+    </command_interface>
+    <state_interface name="position"/>
+    <state_interface name="velocity"/>
+  </joint>
+</ros2_control>
 </robot>
